File: Arduino.sch (KiCad schematic (older format))
At the start: 0 parts

Commit message: Finished Week 3, Unit 10: Revisiting The Current Fan Module
Parts:
- added R? (x15): R, ~, symbol R
- added SHIELD?: ARDUINO_SHIELD, symbol ARDUINO_SHIELD
Connections:
- net MISO: now also R?.2
- net MOSI: now also R?.2
- net RELAY+: now also R?.2
- net SCLK: now also R?.2
- net TACH_MEAS: now also R?.1
- new net: R?.1, SHIELD?.0
- new net: R?.1, SHIELD?.1
- new net: R?.1, SHIELD?.10
- new net: R?.1, SHIELD?.11
- new net: R?.1, SHIELD?.12
- new net: R?.1, SHIELD?.13
- new net: R?.1, SHIELD?.8
- new net: R?.1, SHIELD?.9
- new net: R?.2, SHIELD?.AD0
- new net: R?.2, SHIELD?.AD1
- new net: R?.2, SHIELD?.AD2
- new net: R?.2, SHIELD?.AD3
- new net: R?.2, SHIELD?.V_IN
- new net +12P: R?.1
- new net ADC_CS_N: R?.2
- new net CURR_MEAS: R?.1
- new net DAC_CS_N: R?.2
- new net FAN_MODE: R?.2
- new net FAN_PWM: R?.2
- new net GND: R?.1
- new net LED_EN_PWM: R?.2
- new net RELAY-: R?.2
- new net V+_ADJ_MON: R?.1
- new net V-_ADJ_MON: R?.1
