File: Power.sch (KiCad schematic (older format))
At the start: 11 parts

Commit message: Finished Week 3, Unit 10: Revisiting The Current Fan Module
Parts:
- removed F? (x4): FUSE, ~, symbol FUSE
- added TH? (x4): THERMISTOR, ~, symbol THERMISTOR
Connections:
- net +12P: now also TH?.2
- net +3.3V: now also TH?.2
- net +5V: now also TH?.2
- net -12p: now also TH?.2
- net +12C: now reaches P?.10 (P10)
- net +12C: now also TH?.1
- net at P?.14 (P14): now also TH?.1
- net at P?.2 (P2): now also TH?.1
- net at P?.4 (P4), P?.6 (P6): now also TH?.1
Changed lines of the file:
@@
 LIBS:valves
 LIBS:BenchBudEE
+LIBS:arduino_shieldsNCL
 LIBS:BenchBudEE-cache
 EELAYER 27 0
@@
 $Descr A4 11693 8268
 encoding utf-8
-Sheet 5 9
+Sheet 4 9
 Title ""
-Date "6 feb 2014"
+Date "7 feb 2014"
 Rev ""
 Comp ""
@@
 F 3 "" H 4300 1200 60  0000 C CNN
 	1    4300 1200
-	1    0    0    -1
-$EndComp
-$Comp
-L FUSE F?
-U 1 1 52F23E72
-P 3250 1800
-F 0 "F?" H 3350 1850 40  0000 C CNN
-F 1 "FUSE" H 3150 1750 40  0000 C CNN
-F 2 "~" H 3250 1800 60  0000 C CNN
-F 3 "~" H 3250 1800 60  0000 C CNN
-	1    3250 1800
-	1    0    0    -1
-$EndComp
-$Comp
-L FUSE F?
-U 1 1 52F23E89
-P 3850 2000
-F 0 "F?" H 3950 2050 40  0000 C CNN
-F 1 "FUSE" H 3750 1950 40  0000 C CNN
-F 2 "~" H 3850 2000 60  0000 C CNN
-F 3 "~" H 3850 2000 60  0000 C CNN
-	1    3850 2000
-	1    0    0    -1
-$EndComp
-$Comp
-L FUSE F?
-U 1 1 52F23E93
-P 4350 2200
-F 0 "F?" H 4450 2250 40  0000 C CNN
-F 1 "FUSE" H 4250 2150 40  0000 C CNN
-F 2 "~" H 4350 2200 60  0000 C CNN
-F 3 "~" H 4350 2200 60  0000 C CNN
-	1    4350 2200
-	1    0    0    -1
-$EndComp
-$Comp
-L FUSE F?
-U 1 1 52F23E99
-P 5050 2400
-F 0 "F?" H 5150 2450 40  0000 C CNN
-F 1 "FUSE" H 4950 2350 40  0000 C CNN
-F 2 "~" H 5050 2400 60  0000 C CNN
-F 3 "~" H 5050 2400 60  0000 C CNN
-	1    5050 2400
 	1    0    0    -1
 $EndComp
@@
 	8200 2750 8200 2650
 Connection ~ 7650 2750
+$Comp
+L +12C #PWR?
+U 1 1 52F51751
+P 3000 1200
+F 0 "#PWR?" H 3000 1170 30  0001 C CNN
+F 1 "+12C" H 3000 1310 40  0000 C CNN
+F 2 "" H 3000 1200 60  0000 C CNN
+F 3 "" H 3000 1200 60  0000 C CNN
+	1    3000 1200
+	1    0    0    -1
+$EndComp
+Wire Wire Line
+	3000 1200 3000 2200
+Connection ~ 3000 2200
+$Comp
+L THERMISTOR TH?
+U 1 1 52F51BBD
+P 3250 1800
+F 0 "TH?" V 3350 1850 50  0000 C CNN
+F 1 "THERMISTOR" V 3150 1800 50  0000 C CNN
+F 2 "~" H 3250 1800 60  0000 C CNN
+F 3 "~" H 3250 1800 60  0000 C CNN
+	1    3250 1800
+	0    -1   -1   0
+$EndComp
+$Comp
+L THERMISTOR TH?
+U 1 1 52F51BCA
+P 3850 2000
+F 0 "TH?" V 3950 2050 50  0000 C CNN
+F 1 "THERMISTOR" V 3750 2000 50  0000 C CNN
+F 2 "~" H 3850 2000 60  0000 C CNN
+F 3 "~" H 3850 2000 60  0000 C CNN
+	1    3850 2000
+	0    -1   -1   0
+$EndComp
+$Comp
+L THERMISTOR TH?
+U 1 1 52F51BD0
+P 4350 2200
+F 0 "TH?" V 4450 2250 50  0000 C CNN
+F 1 "THERMISTOR" V 4250 2200 50  0000 C CNN
+F 2 "~" H 4350 2200 60  0000 C CNN
+F 3 "~" H 4350 2200 60  0000 C CNN
+	1    4350 2200
+	0    -1   -1   0
+$EndComp
+$Comp
+L THERMISTOR TH?
+U 1 1 52F51BD6
+P 5050 2400
+F 0 "TH?" V 5150 2450 50  0000 C CNN
+F 1 "THERMISTOR" V 4950 2400 50  0000 C CNN
+F 2 "~" H 5050 2400 60  0000 C CNN
+F 3 "~" H 5050 2400 60  0000 C CNN
+	1    5050 2400
+	0    -1   -1   0
+$EndComp
 $EndSCHEMATC
